File: hardware/ECE49595_Team20_main/ECE49595_Team20_main.kicad_sch (KiCad schematic)
At the start: 0 parts

Commit message: Yashar made me
Other:
- added sheet MCU Main (mcu_main.kicad_sch)
Changed lines of the file:
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@@
 		(company "ECE49595 Team 20")
+	)
+	(sheet
+		(at 25.4 25.4)
+		(size 25.4 25.4)
+		(exclude_from_sim no)
+		(in_bom yes)
+		(on_board yes)
+		(dnp no)
+		(fields_autoplaced yes)
+		(stroke
+			(width 0.1524)
+			(type solid)
+		)
+		(fill
+			(color 0 0 0 0.0000)
+		)
+		(property "Sheetname" "MCU Main"
+			(at 25.4 24.6884 0)
+			(effects
+				(font
+					(size 1.27 1.27)
+				)
+				(justify left bottom)
+			)
+		)
+		(property "Sheetfile" "mcu_main.kicad_sch"
+			(at 25.4 51.3846 0)
+			(effects
+				(font
+					(size 1.27 1.27)
+				)
+				(justify left top)
+			)
+		)
+		(instances
+			(project "ECE49595_Team20_main"
+				(path "/cbe9655e-6153-4339-aa3b-1ea5dc7d3b3f"
+					(page "2")
+				)
+			)
+		)
 	)
 	(sheet_instances
